File: schema/espurna.brd (EAGLE design)
At the start: 50 x 50 mm, 23 parts, among them IC1 ESP-12-SMD, IC2 AMS1117-3.3

Commit message: Improved board layout
Parts:
- moved VARISTOR 2.16 mm to (12.6, 32.4)
Routing:
- net NC: track 23.7 -> 47.4 mm
- net LINE: track 29.7 -> 44.1 mm
- net NO: track 9.83 -> 19.7 mm
- net N$8: track 20.5 -> 18.4 mm
Other:
- outline, holes or cut-outs redrawn
